File: currentsensor/board/schematic.sch (EAGLE design)
At the start: 41 parts, among them IC1 4050D

Commit message: layout
Connections:
- net SCL: now also I2C.2; no longer I2C.1
- net SDA: now also I2C.1; no longer I2C.2
Other:
- moved on the sheet: I2C
Changed lines of the file:
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@@
 <instance part="C3" gate="G$1" x="-27.94" y="106.68"/>
 <instance part="C4" gate="G$1" x="-20.32" y="106.68"/>
-<instance part="I2C" gate="G$1" x="226.06" y="-109.22" rot="R180"/>
-<instance part="GND17" gate="1" x="215.9" y="-119.38"/>
+<instance part="I2C" gate="G$1" x="231.14" y="-106.68" rot="R180"/>
+<instance part="GND17" gate="1" x="220.98" y="-119.38"/>
 <instance part="R14" gate="G$1" x="208.28" y="-91.44" rot="R270"/>
 <instance part="R17" gate="G$1" x="218.44" y="-91.44" rot="R270"/>
@@
 <segment>
 <pinref part="I2C" gate="G$1" pin="3"/>
-<wire x1="218.44" y1="-111.76" x2="215.9" y2="-111.76" width="0.1524" layer="91"/>
-<wire x1="215.9" y1="-111.76" x2="215.9" y2="-116.84" width="0.1524" layer="91"/>
+<wire x1="223.52" y1="-109.22" x2="220.98" y2="-109.22" width="0.1524" layer="91"/>
+<wire x1="220.98" y1="-109.22" x2="220.98" y2="-116.84" width="0.1524" layer="91"/>
 <pinref part="GND17" gate="1" pin="GND"/>
 </segment>
@@
 </segment>
 <segment>
-<pinref part="I2C" gate="G$1" pin="2"/>
-<wire x1="218.44" y1="-109.22" x2="208.28" y2="-109.22" width="0.1524" layer="91"/>
-<label x="137.16" y="-109.22" size="1.778" layer="95" rot="R180" xref="yes"/>
+<label x="134.62" y="-104.14" size="1.778" layer="95" rot="R180" xref="yes"/>
 <pinref part="R14" gate="G$1" pin="2"/>
-<wire x1="208.28" y1="-109.22" x2="139.7" y2="-109.22" width="0.1524" layer="91"/>
-<wire x1="139.7" y1="-109.22" x2="137.16" y2="-109.22" width="0.1524" layer="91"/>
-<wire x1="208.28" y1="-109.22" x2="208.28" y2="-96.52" width="0.1524" layer="91"/>
-<junction x="208.28" y="-109.22"/>
+<wire x1="208.28" y1="-104.14" x2="139.7" y2="-104.14" width="0.1524" layer="91"/>
+<wire x1="139.7" y1="-104.14" x2="134.62" y2="-104.14" width="0.1524" layer="91"/>
+<wire x1="208.28" y1="-104.14" x2="208.28" y2="-96.52" width="0.1524" layer="91"/>
 <pinref part="U$5" gate="G$1" pin="SDA"/>
 <wire x1="154.94" y1="-86.36" x2="139.7" y2="-86.36" width="0.1524" layer="91"/>
-<wire x1="139.7" y1="-86.36" x2="139.7" y2="-109.22" width="0.1524" layer="91"/>
-<junction x="139.7" y="-109.22"/>
+<wire x1="139.7" y1="-86.36" x2="139.7" y2="-104.14" width="0.1524" layer="91"/>
+<junction x="139.7" y="-104.14"/>
+<pinref part="I2C" gate="G$1" pin="1"/>
+<wire x1="223.52" y1="-104.14" x2="208.28" y2="-104.14" width="0.1524" layer="91"/>
+<junction x="208.28" y="-104.14"/>
 </segment>
 </net>
@@
 </segment>
 <segment>
-<label x="132.08" y="-106.68" size="1.778" layer="95" rot="R180" xref="yes"/>
-<pinref part="I2C" gate="G$1" pin="1"/>
-<wire x1="218.44" y1="-106.68" x2="137.16" y2="-106.68" width="0.1524" layer="91"/>
-<pinref part="R17" gate="G$1" pin="2"/>
-<wire x1="218.44" y1="-106.68" x2="218.44" y2="-96.52" width="0.1524" layer="91"/>
-<junction x="218.44" y="-106.68"/>
-<wire x1="132.08" y1="-106.68" x2="137.16" y2="-106.68" width="0.1524" layer="91"/>
+<label x="127" y="-106.68" size="1.778" layer="95" rot="R180" xref="yes"/>
+<wire x1="127" y1="-106.68" x2="137.16" y2="-106.68" width="0.1524" layer="91"/>
 <wire x1="137.16" y1="-106.68" x2="137.16" y2="-83.82" width="0.1524" layer="91"/>
 <pinref part="U$5" gate="G$1" pin="SCL"/>
 <wire x1="137.16" y1="-83.82" x2="154.94" y2="-83.82" width="0.1524" layer="91"/>
+<pinref part="I2C" gate="G$1" pin="2"/>
+<wire x1="137.16" y1="-106.68" x2="218.44" y2="-106.68" width="0.1524" layer="91"/>
+<pinref part="R17" gate="G$1" pin="2"/>
+<wire x1="218.44" y1="-106.68" x2="223.52" y2="-106.68" width="0.1524" layer="91"/>
+<wire x1="218.44" y1="-96.52" x2="218.44" y2="-106.68" width="0.1524" layer="91"/>
 <junction x="137.16" y="-106.68"/>
-</segment>
-</net>
+<junction x="218.44" y="-106.68"/>
+</segment>
+</net>

Commit message: layout
Parts:
- added PCB1: PCB_DP_RECTANGLE-50X75, dp_pcb:PCB_DP_RECTANGLE-50X75
Changed lines of the file:
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@@
 <part name="GND20" library="supply1" deviceset="GND" device=""/>
 <part name="GND21" library="supply1" deviceset="GND" device=""/>
+<part name="PCB1" library="dp_pcb" deviceset="PCB_DP_RECTANGLE" device="-50X75"/>
 </parts>
 <sheets>
@@
 <instance part="GND20" gate="1" x="185.42" y="-99.06"/>
 <instance part="GND21" gate="1" x="195.58" y="-99.06"/>
+<instance part="PCB1" gate="G$1" x="-22.86" y="-40.64"/>
 </instances>
 <busses>

Commit message: layout
Parts:
- removed SWITCH: (no value), con-lstb:MA03-1
- added JP1: (no value), pinhead:PINHD-1X2
Connections:
- removed net SWITCH2: SWITCH.2
- net 5V_ACT: now also CON-LT.4; no longer CON-LB.1
- net GND: now also JP1.1; no longer SWITCH.1
- net SWITCH: now also CON-LB.1, JP1.2; no longer CON-LT.2, SWITCH.3
- net TFT_DC: now also CON-LT.3; no longer CON-LT.4
- net TFT_RST: now also CON-LT.2; no longer CON-LT.3
Changed lines of the file:
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@@
 <part name="U$3" library="custom_devices" deviceset="BSS83P" device=""/>
 <part name="R8" library="resistor" deviceset="R-EU_" device="R1206" value="39k"/>
-<part name="SWITCH" library="con-lstb" deviceset="MA03-1" device=""/>
 <part name="SV2" library="con-lstb" deviceset="MA07-2" device=""/>
 <part name="E1" library="ble" deviceset="HM-10" device="-BOARD"/>
@@
 <part name="GND21" library="supply1" deviceset="GND" device=""/>
 <part name="PCB1" library="dp_pcb" deviceset="PCB_DP_RECTANGLE" device="-50X75"/>
+<part name="JP1" library="pinhead" deviceset="PINHD-1X2" device=""/>
 </parts>
 <sheets>
@@
 <instance part="U$3" gate="G$1" x="193.04" y="93.98"/>
 <instance part="R8" gate="G$1" x="185.42" y="104.14" rot="R180"/>
-<instance part="SWITCH" gate="G$1" x="139.7" y="109.22" rot="R180"/>
 <instance part="SV2" gate="G$1" x="139.7" y="71.12"/>
 <instance part="E1" gate="G$1" x="27.94" y="-58.42"/>
@@
 <instance part="GND21" gate="1" x="195.58" y="-99.06"/>
 <instance part="PCB1" gate="G$1" x="-22.86" y="-40.64"/>
+<instance part="JP1" gate="G$1" x="142.24" y="109.22"/>
 </instances>
 <busses>
@@
 </segment>
 <segment>
-<pinref part="SWITCH" gate="G$1" pin="1"/>
-<wire x1="132.08" y1="111.76" x2="127" y2="111.76" width="0.1524" layer="91"/>
 <label x="127" y="111.76" size="1.778" layer="95" rot="R180" xref="yes"/>
+<pinref part="JP1" gate="G$1" pin="1"/>
+<wire x1="139.7" y1="111.76" x2="127" y2="111.76" width="0.1524" layer="91"/>
 </segment>
 <segment>
@@
 <net name="SWITCH" class="0">
 <segment>
-<pinref part="SWITCH" gate="G$1" pin="3"/>
-<wire x1="132.08" y1="106.68" x2="127" y2="106.68" width="0.1524" layer="91"/>
-<label x="127" y="106.68" size="1.778" layer="95" rot="R180" xref="yes"/>
-</segment>
-<segment>
-<pinref part="CON-LT" gate="1" pin="2"/>
-<wire x1="-20.32" y1="-5.08" x2="-15.24" y2="-5.08" width="0.1524" layer="91"/>
-<label x="-15.24" y="-5.08" size="1.778" layer="95" xref="yes"/>
+<label x="119.38" y="109.22" size="1.778" layer="95" rot="R180" xref="yes"/>
+<pinref part="JP1" gate="G$1" pin="2"/>
+<wire x1="139.7" y1="109.22" x2="119.38" y2="109.22" width="0.1524" layer="91"/>
+</segment>
+<segment>
+<pinref part="CON-LB" gate="G$1" pin="1"/>
+<wire x1="-20.32" y1="-30.48" x2="-15.24" y2="-30.48" width="0.1524" layer="91"/>
+<label x="-15.24" y="-30.48" size="1.778" layer="95" xref="yes"/>
 </segment>
 </net>
@@
 </segment>
 <segment>
-<pinref part="CON-LB" gate="G$1" pin="1"/>
-<wire x1="-20.32" y1="-30.48" x2="-15.24" y2="-30.48" width="0.1524" layer="91"/>
-<label x="-15.24" y="-30.48" size="1.778" layer="95" xref="yes"/>
+<pinref part="CON-LT" gate="1" pin="4"/>
+<wire x1="-20.32" y1="0" x2="-15.24" y2="0" width="0.1524" layer="91"/>
+<label x="-15.24" y="0" size="1.778" layer="95" xref="yes"/>
 </segment>
 </net>
@@
 </segment>
 </net>
-<net name="SWITCH2" class="0">
-<segment>
-<label x="119.38" y="109.22" size="1.778" layer="95" rot="R180" xref="yes"/>
-<pinref part="SWITCH" gate="G$1" pin="2"/>
-<wire x1="132.08" y1="109.22" x2="119.38" y2="109.22" width="0.1524" layer="91"/>
-<junction x="132.08" y="109.22"/>
-</segment>
-</net>
 <net name="TFT_CS" class="0">
 <segment>
@@
 </segment>
 <segment>
+<pinref part="CON-LT" gate="1" pin="2"/>
+<wire x1="-20.32" y1="-5.08" x2="-15.24" y2="-5.08" width="0.1524" layer="91"/>
+<label x="-15.24" y="-5.08" size="1.778" layer="95" xref="yes"/>
+</segment>
+</net>
+<net name="TOUCH_IRQ" class="0">
+<segment>
+<pinref part="SV2" gate="G$1" pin="12"/>
+<wire x1="132.08" y1="76.2" x2="129.54" y2="76.2" width="0.1524" layer="91"/>
+<label x="129.54" y="76.2" size="1.778" layer="95" rot="R180" xref="yes"/>
+</segment>
+<segment>
+<pinref part="CON-LB" gate="G$1" pin="4"/>
+<wire x1="-20.32" y1="-22.86" x2="2.54" y2="-22.86" width="0.1524" layer="91"/>
+<label x="2.54" y="-22.86" size="1.778" layer="95" xref="yes"/>
+</segment>
+</net>
+<net name="TOUCH_CS" class="0">
+<segment>
+<pinref part="SV2" gate="G$1" pin="11"/>
+<wire x1="147.32" y1="76.2" x2="152.4" y2="76.2" width="0.1524" layer="91"/>
+<label x="152.4" y="76.2" size="1.778" layer="95" xref="yes"/>
+</segment>
+<segment>
+<pinref part="CON-LB" gate="G$1" pin="5"/>
+<wire x1="-20.32" y1="-20.32" x2="-15.24" y2="-20.32" width="0.1524" layer="91"/>
+<label x="-15.24" y="-20.32" size="1.778" layer="95" xref="yes"/>
+</segment>
+</net>
+<net name="TFT_LED" class="0">
+<segment>
+<pinref part="SV2" gate="G$1" pin="9"/>
+<wire x1="147.32" y1="73.66" x2="167.64" y2="73.66" width="0.1524" layer="91"/>
+<label x="167.64" y="73.66" size="1.778" layer="95" xref="yes"/>
+</segment>
+<segment>
+<pinref part="CON-LB" gate="G$1" pin="2"/>
+<wire x1="-20.32" y1="-27.94" x2="2.54" y2="-27.94" width="0.1524" layer="91"/>
+<label x="2.54" y="-27.94" size="1.778" layer="95" xref="yes"/>
+</segment>
+</net>
+<net name="TFT_DC" class="0">
+<segment>
+<pinref part="SV2" gate="G$1" pin="7"/>
+<wire x1="147.32" y1="71.12" x2="152.4" y2="71.12" width="0.1524" layer="91"/>
+<label x="152.4" y="71.12" size="1.778" layer="95" xref="yes"/>
+</segment>
+<segment>
 <pinref part="CON-LT" gate="1" pin="3"/>
 <wire x1="-20.32" y1="-2.54" x2="0" y2="-2.54" width="0.1524" layer="91"/>
@@
 </segment>
 </net>
-<net name="TOUCH_IRQ" class="0">
-<segment>
-<pinref part="SV2" gate="G$1" pin="12"/>
-<wire x1="132.08" y1="76.2" x2="129.54" y2="76.2" width="0.1524" layer="91"/>
-<label x="129.54" y="76.2" size="1.778" layer="95" rot="R180" xref="yes"/>
-</segment>
-<segment>
-<pinref part="CON-LB" gate="G$1" pin="4"/>
-<wire x1="-20.32" y1="-22.86" x2="2.54" y2="-22.86" width="0.1524" layer="91"/>
-<label x="2.54" y="-22.86" size="1.778" layer="95" xref="yes"/>
-</segment>
-</net>
-<net name="TOUCH_CS" class="0">
-<segment>
-<pinref part="SV2" gate="G$1" pin="11"/>
-<wire x1="147.32" y1="76.2" x2="152.4" y2="76.2" width="0.1524" layer="91"/>
-<label x="152.4" y="76.2" size="1.778" layer="95" xref="yes"/>
-</segment>
-<segment>
-<pinref part="CON-LB" gate="G$1" pin="5"/>
-<wire x1="-20.32" y1="-20.32" x2="-15.24" y2="-20.32" width="0.1524" layer="91"/>
-<label x="-15.24" y="-20.32" size="1.778" layer="95" xref="yes"/>
-</segment>
-</net>
-<net name="TFT_LED" class="0">
-<segment>
-<pinref part="SV2" gate="G$1" pin="9"/>
-<wire x1="147.32" y1="73.66" x2="167.64" y2="73.66" width="0.1524" layer="91"/>
-<label x="167.64" y="73.66" size="1.778" layer="95" xref="yes"/>
-</segment>
-<segment>
-<pinref part="CON-LB" gate="G$1" pin="2"/>
-<wire x1="-20.32" y1="-27.94" x2="2.54" y2="-27.94" width="0.1524" layer="91"/>
-<label x="2.54" y="-27.94" size="1.778" layer="95" xref="yes"/>
-</segment>
-</net>
-<net name="TFT_DC" class="0">
-<segment>
-<pinref part="SV2" gate="G$1" pin="7"/>
-<wire x1="147.32" y1="71.12" x2="152.4" y2="71.12" width="0.1524" layer="91"/>
-<label x="152.4" y="71.12" size="1.778" layer="95" xref="yes"/>
-</segment>
-<segment>
-<pinref part="CON-LT" gate="1" pin="4"/>
-<wire x1="-20.32" y1="0" x2="-15.24" y2="0" width="0.1524" layer="91"/>
-<label x="-15.24" y="0" size="1.778" layer="95" xref="yes"/>
-</segment>
-</net>

Commit message: layout finished
Parts:
- removed JP1: (no value), pinhead:PINHD-1X2
- removed SV2: (no value), con-lstb:MA07-2
- added BUTTON: (no value), pinhead:PINHD-1X2
- added DISPLAY: (no value), con-lstb:MA07-2
- added R13: 39k, resistor:R-EU_R1206
- C5, C6: value 10nF -> 7pF
- R6, R7: value 4k7 -> 680
Connections:
- removed net SWITCH: CON-LB.1, JP1.2
- new net BUTTON: BUTTON.2, CON-LB.1
- net +3V3: now also R13.1
- net BLE_RESET: now also IC1A.I; no longer IC1C.I
- net GND: now also BUTTON.1, DISPLAY.13, DISPLAY.14, DISPLAY.2; no longer JP1.1, SV2.13, SV2.14, SV2.2
- net LCD_5V: now also DISPLAY.1; no longer SV2.1
- net N$11: now also IC1C.O; no longer IC1A.O
- net N$12: now also IC1A.O; no longer IC1C.O
- net SD_CS: now also DISPLAY.10; no longer SV2.10
- net SPI_CLK: now also DISPLAY.3; no longer SV2.3
- net SPI_MISO: now also DISPLAY.4, R13.2; no longer SV2.4
- net SPI_MOSI: now also DISPLAY.5; no longer SV2.5
- net TFT_CS: now also DISPLAY.6; no longer SV2.6
- net TFT_DC: now also DISPLAY.7; no longer SV2.7
- net TFT_LED: now also DISPLAY.9; no longer SV2.9
- net TFT_RST: now also DISPLAY.8; no longer SV2.8
- net TOUCH_CS: now also DISPLAY.11; no longer SV2.11
- net TOUCH_IRQ: now also DISPLAY.12; no longer SV2.12
- net UART_TX: now also IC1C.I; no longer IC1A.I
Other:
- moved on the sheet: IC1A, IC1C, R8, U$3
