File: currentsensor/board/schematic.brd (EAGLE design)
At the start: 49.5 x 49.4 mm, 41 parts, among them IC1 4050D

Commit message: layout
Parts:
- moved C5 57.0 mm to (1.82, 38.1), turned to 270 degrees
- moved IC1 46.7 mm to (3.44, 57.1), flipped to the bottom
- moved C6 43.0 mm to (1.68, 14.5)
- moved R10 36.3 mm to (2.85, 22.1)
- moved C1 31.3 mm to (3.93, 34.1), turned to 180 degrees
- moved E1 31.3 mm to (80.5, 34.7), flipped to the bottom
- moved Q1 27.5 mm to (79.7, 59.9), turned to 90 degrees
- moved I2C 25.5 mm to (30.8, 70.1)
- moved R17 24.5 mm to (33.4, 63.6)
- moved R14 23.9 mm to (28.2, 63.6)
- moved C2 22.1 mm to (3.27, 28.5), turned to 180 degrees
- moved U$5 8.46 mm to (30.3, 46.5), flipped to the bottom
- moved SV2 2.38 mm to (16.0, 41.7)
Connections:
- net SCL: now also I2C.2; no longer I2C.1
- net SDA: now also I2C.1; no longer I2C.2
Routing:
- net GND: track 105.0 -> 29.2 mm, vias 7 -> 5
- net SPI_CLK: track 0.03 -> 40.9 mm
- net SCL: track 10.7 -> 42.8 mm, vias 0 -> 2
- net +5V: track 93.6 -> 62.5 mm
- net SPI_MISO: track 7.64 -> 36.6 mm
- net SPI_MOSI: track 5.21 -> 31.0 mm
- net U_LOAD: track 112.9 -> 90.9 mm, vias 5 -> 4
- net TFT_LED: track 0.00 -> 17.0 mm
- net TFT_CS: track 7.82 -> 24.2 mm
- net RTC_IRQ: track 9.24 -> 24.9 mm
- net SDA: track 15.6 -> 28.9 mm
- net LCD_5V: track 16.9 -> 24.8 mm
- net SWITCH: track 11.4 -> 5.64 mm
- net SD_CS: track 0.76 -> 6.25 mm
- net UART_TX: track 4.58 -> 0.00 mm, vias 1 -> 0
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
Commit message: layout
Parts:
- added PCB1: PCB_DP_RECTANGLE-50X75, dp_pcb:DP5075_V1
- moved C6 72.0 mm to (54.3, 63.6), turned to 90 degrees
- moved C2 69.0 mm to (61.9, 65.0)
- moved C1 59.1 mm to (60.1, 52.5)
- moved C5 56.0 mm to (54.3, 57.4)
- moved IC1 47.1 mm to (48.8, 44.3)
- moved E1 35.7 mm to (53.4, 57.8), turned to 270 degrees
- moved U$5 34.1 mm to (61.9, 59.3), flipped to the top, turned to 270 degrees
- moved R10 33.9 mm to (31.0, 41.0), turned to 90 degrees
- moved C3 32.8 mm to (77.0, 54.0), turned to 90 degrees
- moved Q1 28.4 mm to (51.4, 60.5)
- moved C4 28.2 mm to (73.3, 53.9), turned to 90 degrees
- moved C7 28.2 mm to (68.9, 53.8), turned to 90 degrees
- moved X1 28.0 mm to (75.4, 39.7)
- moved G1 8.45 mm to (65.0, 39.6), turned to 0 degrees
- moved U$3 4.75 mm to (17.3, 60.1)
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Routing:
- net GND: track 29.2 -> 137.2 mm, vias 5 -> 4
- net RTC_IRQ: track 24.9 -> 85.8 mm
- net SDA: track 28.9 -> 74.4 mm
- net +5V: track 62.5 -> 106.6 mm
- net SCL: track 42.8 -> 74.5 mm
- net VBAK: track 0.00 -> 31.0 mm, vias 0 -> 1
- net N$17: track 0.00 -> 8.07 mm
- net N$16: track 0.00 -> 8.06 mm
- net LCD_5V: track 24.8 -> 20.1 mm
- net SPI_CLK: track 40.9 -> 36.8 mm
- net SPI_MISO: track 36.6 -> 32.9 mm
- net SPI_MOSI: track 31.0 -> 27.6 mm
- net SENSE_LOAD: track 46.0 -> 43.4 mm, vias 1 -> 0
- net ADC_I_DISCH: track 9.62 -> 12.2 mm
- net TFT_CS: track 24.2 -> 21.6 mm
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- removed copper zone on layer 1, net GND
- removed copper zone on layer 16, net GND
Other:
- board size 49.5 x 49.4 mm -> 75 x 50 mm

Commit message: layout
Parts:
- removed SWITCH: (no value), con-lstb:MA03-1
- added JP1: (no value), pinhead:1X02
- moved U$3 21.6 mm to (27.3, 41.0)
- moved R8 18.6 mm to (30.9, 41.0), turned to 270 degrees
- moved I2C 4.18 mm to (30.8, 65.9)
- moved R14 3.78 mm to (28.2, 59.8)
- moved R17 3.78 mm to (33.4, 59.8)
- moved R10 3.20 mm to (34.2, 41.0)
- moved SV2 2.18 mm to (14.7, 43.5)
- moved C7 1.66 mm to (70.5, 53.6)
- moved C3 1.66 mm to (78.7, 53.8)
- moved C4 1.66 mm to (74.9, 53.7)
- moved X1 1.66 mm to (77.1, 39.7)
- moved OW 0.14 mm to (30.8, 25.9)
Connections:
- removed net SWITCH2: SWITCH.2
- net 5V_ACT: now also CON-LT.4; no longer CON-LB.1
- net GND: now also JP1.1; no longer SWITCH.1
- net SWITCH: now also CON-LB.1, JP1.2; no longer CON-LT.2, SWITCH.3
- net TFT_DC: now also CON-LT.3; no longer CON-LT.4
- net TFT_RST: now also CON-LT.2; no longer CON-LT.3
Routing:
- net GND: track 137.2 -> 272.4 mm, vias 4 -> 6
- net RTC_IRQ: track 85.8 -> 20.5 mm, vias 0 -> 1
- net U_LOAD: track 91.8 -> 113.7 mm, vias 2 -> 3
- net +5V: track 106.6 -> 124.3 mm, vias 2 -> 4
- net 5V_ACT: track 27.8 -> 14.0 mm
- net SPI_MISO: track 32.9 -> 44.9 mm
- net SPI_CLK: track 36.8 -> 47.4 mm
- net SWITCH: track 5.64 -> 10.5 mm
- net TOUCH_IRQ: track 7.28 -> 10.5 mm
- net TFT_LED: track 17.0 -> 19.8 mm
- net SPI_MOSI: track 27.6 -> 30.3 mm
- net SCL: track 74.5 -> 77.2 mm, vias 2 -> 0
- net SDA: track 74.4 -> 76.9 mm
- net TFT_CS: track 21.6 -> 23.9 mm
- net SD_CS: track 6.25 -> 8.29 mm
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
Commit message: layout finished
Parts:
- removed JP1: (no value), pinhead:1X02
- removed SV2: (no value), con-lstb:MA07-2
- added BUTTON: (no value), pinhead:1X02
- added DISPLAY: (no value), con-lstb:MA07-2
- added R13: 39k, resistor:R1206
- C5, C6: value 10nF -> 7pF
- R6, R7: value 4k7 -> 680
- moved E1 25.8 mm to (52.8, 32.0), turned to 180 degrees
- moved IC1 20.2 mm to (51.9, 64.2), turned to 0 degrees
- moved Q1 17.7 mm to (69.0, 62.1), turned to 270 degrees
- moved C5 14.0 mm to (66.1, 65.0), turned to 90 degrees
- moved C6 12.7 mm to (66.1, 58.8), turned to 270 degrees
- moved C2 8.29 mm to (58.6, 57.4), turned to 0 degrees
- moved U$5 5.13 mm to (58.6, 63.1), turned to 90 degrees
- moved R17 1.61 mm to (31.8, 59.8)
- moved OW 1.61 mm to (29.2, 25.9)
- moved R11 1.61 mm to (29.3, 32.9)
- moved R8 1.61 mm to (29.3, 41.0)
- moved U$3 1.61 mm to (25.7, 41.0)
- moved U$4 1.61 mm to (25.7, 30.2)
- moved CON-LB 1.61 mm to (21.6, 30.8)
- moved CON-LT 1.61 mm to (21.6, 52.3)
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Connections:
- removed net SWITCH: CON-LB.1, JP1.2
- new net BUTTON: BUTTON.2, CON-LB.1
- net +3V3: now also R13.1
- net BLE_RESET: now also IC1.3; no longer IC1.7
- net GND: now also BUTTON.1, DISPLAY.13, DISPLAY.14, DISPLAY.2; no longer JP1.1, SV2.13, SV2.14, SV2.2
- net LCD_5V: now also DISPLAY.1; no longer SV2.1
- net N$11: now also IC1.6; no longer IC1.2
- net N$12: now also IC1.2; no longer IC1.6
- net SD_CS: now also DISPLAY.10; no longer SV2.10
- net SPI_CLK: now also DISPLAY.3; no longer SV2.3
- net SPI_MISO: now also DISPLAY.4, R13.2; no longer SV2.4
- net SPI_MOSI: now also DISPLAY.5; no longer SV2.5
- net TFT_CS: now also DISPLAY.6; no longer SV2.6
- net TFT_DC: now also DISPLAY.7; no longer SV2.7
- net TFT_LED: now also DISPLAY.9; no longer SV2.9
- net TFT_RST: now also DISPLAY.8; no longer SV2.8
- net TOUCH_CS: now also DISPLAY.11; no longer SV2.11
- net TOUCH_IRQ: now also DISPLAY.12; no longer SV2.12
- net UART_TX: now also IC1.7; no longer IC1.3
- net U_LOAD: now also U$1.6, U$2.6; no longer U$1.5, U$2.5
Routing:
- net GND: track 272.4 -> 354.6 mm, vias 6 -> 5
- net +3V3: track 0.00 -> 72.0 mm, vias 0 -> 2
- net UART_RX: track 0.00 -> 56.8 mm
- net U_LOAD: track 113.7 -> 166.1 mm, vias 3 -> 4
- net RTC_IRQ: track 20.5 -> 65.9 mm, vias 1 -> 2
- net BLE_RESET: track 0.00 -> 39.7 mm, vias 0 -> 2
- net N$10: track 0.00 -> 37.3 mm
- net N$11: track 0.00 -> 36.9 mm
- net UART_RTS: track 0.00 -> 34.1 mm, vias 0 -> 2
- net SPI_MISO: track 44.9 -> 78.6 mm
- net UART_TX: track 0.00 -> 32.6 mm
- net N$12: track 0.00 -> 26.1 mm
- net SDA: track 76.9 -> 52.8 mm
- net SCL: track 77.2 -> 57.5 mm
- net BUTTON: track 0.00 -> 10.5 mm
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- added copper zone on layer 1, net GND
- added copper zone on layer 16, net GND
Other:
- board text added: "+5V"
- board text added: "DATA"
- board text added: "RESET"
- board text added: "SCL"
- board text added: "SDA"
- board text removed: "1"

Commit message: layout
Parts:
- moved DISPLAY 3.89 mm to (13.1, 49.7)
Routing:
- net GND: track 354.6 -> 360.8 mm
- net TFT_LED: track 26.3 -> 30.1 mm
- net TFT_CS: track 21.8 -> 17.9 mm
- net TOUCH_IRQ: track 13.4 -> 17.3 mm
- net SPI_MOSI: track 28.0 -> 24.1 mm
- net SPI_CLK: track 47.2 -> 43.3 mm
- net SD_CS: track 11.4 -> 15.3 mm
- net TOUCH_CS: track 13.2 -> 17.0 mm
- net TFT_DC: track 13.9 -> 17.7 mm
- net TFT_RST: track 11.4 -> 15.2 mm
- net LCD_5V: track 22.8 -> 25.9 mm
- net SPI_MISO: track 78.6 -> 77.6 mm
